File: Hardware/Synthesizer.kicad_pcb (KiCad board)
At the start: 2 copper layers, 67 parts, among them J1 MUX_OUT, J2 REF_IN, J3 RFOUTA, J4 RFOUTB, T1 HB-TCM2-63WX+, T2 HB-TCM2-63WX+, U2 74LCX07, U3 GM1207ACPZ-3.3, X1 IQXO-70

Commit message: Nearing completion on schematic and layout.  Ready for design review.
Parts:
- removed R12, R8, R9: 5K1, Resistor_SMD:R_0402_1005Metric
- removed R13: 0, Resistor_SMD:R_0402_1005Metric
- removed R14, R15: NP, Resistor_SMD:R_0402_1005Metric
- added C34: 2.2u, Synthesizer:Cap_0402, F.Cu at (154.4, 103.1)
- added C35: 2.2u, Synthesizer:Cap_0402, F.Cu at (149.1, 103.1)
- added C36: 2.2u, Synthesizer:Cap_0402, F.Cu at (167.4, 97.4)
- added C37: 2.2u, Synthesizer:Cap_0402, F.Cu at (173.0, 97.4)
- added C38: 2.2u, Synthesizer:Cap_0402, F.Cu at (185.0, 88.0)
- added C39: 2.2u, Synthesizer:Cap_0402, F.Cu at (179.7, 88.0)
- added C40: 2.2u, Synthesizer:Cap_0402, F.Cu at (146.8, 90.0)
- added C41: 2.2u, Synthesizer:Cap_0402, F.Cu at (152.3, 90.0)
- added C42: .1u, Synthesizer:Cap_0402, F.Cu at (139.0, 91.5)
- added C43: 47p, Synthesizer:Cap_0402, F.Cu at (139.6, 106.4)
- added C44: .1u, Synthesizer:Cap_0402, F.Cu at (133.0, 102.8)
- added C45: 47p, Synthesizer:Cap_0402, F.Cu at (137.6, 106.4)
- added C46: .1u, Synthesizer:Cap_0402, F.Cu at (140.7, 104.2)
- added C47: .1u, Synthesizer:Cap_0402, F.Cu at (147.7, 83.4)
- added C48: 6.8u, Capacitor_SMD:C_0603_1608Metric, F.Cu at (149.2, 83.7)
- added D2: MM3Z3V6, Diode_SMD:D_SOD-323, F.Cu at (136.9, 108.0)
- added D3: White, LED_SMD:LED_0402_1005Metric, F.Cu at (133.0, 103.9)
- added D4: MM3Z3V6, Diode_SMD:D_SOD-323, F.Cu at (140.2, 108.0)
- added D5: White, LED_SMD:LED_0402_1005Metric, F.Cu at (138.9, 93.1)
- added D6: Yellow, LED_SMD:LED_0402_1005Metric, F.Cu at (142.9, 103.1)
- added D7: Yellow, LED_SMD:LED_0402_1005Metric, F.Cu at (134.8, 103.7)
- added FB1: FerriteBead_Small, Inductor_SMD:L_0805_2012Metric, F.Cu at (134.0, 107.7)
- added J5: USB-C 2.0 16P, Connector_USB:USB_C_Receptacle_G-Switch_GT-USB-7010ASV, F.Cu at (138.5, 114.5)
- added J7: Header 1x3, Connector_PinHeader_2.54mm:PinHeader_1x03_P2.54mm_Vertical, F.Cu at (133.8, 92.9)
- added J8: Screw_Terminal_01x12, TerminalBlock_TE-Connectivity:TerminalBlock_TE_282834-2_1x02_P2.54mm_Horizontal, F.Cu at (133.6, 84.3)
- added R24: 22, Synthesizer:Res_0402, F.Cu at (139.0, 104.9)
- added R25: 22, Synthesizer:Res_0402, F.Cu at (138.0, 104.9)
- added R26: 1K, Synthesizer:Res_0402, F.Cu at (138.9, 94.2)
- added R27: 1K, Synthesizer:Res_0402, F.Cu at (142.9, 100.9)
- added R28: 1K, Synthesizer:Res_0402, F.Cu at (136.4, 104.2)
- added R29: 1K, Synthesizer:Res_0402, F.Cu at (136.6, 96.3)
- added R30: 1K, Synthesizer:Res_0402, F.Cu at (136.1, 93.4)
- added U4: GM1207ACPZ-3.3, Package_TO_SOT_SMD:SOT-23-5, F.Cu at (151.8, 103.5)
- added U5: GM1207ACPZ-3.3, Package_TO_SOT_SMD:SOT-23-5, F.Cu at (170.0, 96.9)
- added U6: GM1207ACPZ-3.3, Package_TO_SOT_SMD:SOT-23-5, F.Cu at (182.4, 87.5)
- added U7: GM1207ACPZ-3.3, Package_TO_SOT_SMD:SOT-23-5, F.Cu at (149.6, 90.5)
- added U8: ATtiny1616-M, Package_DFN_QFN:VQFN-20-1EP_3x3mm_P0.4mm_EP1.7x1.7mm, F.Cu at (142.2, 91.5)
- added U9: FT231XQ, Package_DFN_QFN:QFN-20-1EP_4x4mm_P0.5mm_EP2.5x2.5mm, F.Cu at (138.3, 100.9)
- C1, C10, C11, C12, C13, C14, C15, C16, C17, C18, C19, C2, C20, C21, C22, C23, C24, C25, C27, C28, C29, C3, C30, C31, C32, C33, C4, C5, C6, C7, C8, C9: footprint Capacitor_SMD:C_0402_1005Metric -> Synthesizer:Cap_0402
- C26: value NP -> 330n 25V; footprint Capacitor_SMD:C_0402_1005Metric -> Capacitor_SMD:C_0603_1608Metric
- D1: value LOCK -> D_Schottky; footprint LED_SMD:LED_0402_1005Metric -> Diode_SMD:D_0603_1608Metric
- J1: value MUX_OUT -> REF Select; footprint Connector_Coaxial:SMA_Samtec_SMA-J-P-H-ST-EM1_EdgeMount -> Connector_PinHeader_2.54mm:PinHeader_1x03_P2.54mm_Vertical
- R1, R16, R17, R18, R19, R2, R20, R21, R22, R23, R3, R4, R5, R6: footprint Resistor_SMD:R_0402_1005Metric -> Synthesizer:Res_0402
- R10: value NP -> 5K1; footprint Resistor_SMD:R_0402_1005Metric -> Synthesizer:Res_0402
- R11: value NP -> 1K; footprint Resistor_SMD:R_0402_1005Metric -> Synthesizer:Res_0402
- R7: value OPEN -> 5K1; footprint Resistor_SMD:R_0402_1005Metric -> Synthesizer:Res_0402
- U2: value 74LCX07 -> MC78L05_SOT89; footprint Package_SO:TSSOP-14_4.4x5mm_P0.65mm -> Package_TO_SOT_SMD:SOT-89-3
- moved X1 80.8 mm to (173.2, 85.8), turned to 180 degrees
- moved J2 52.9 mm to (182.0, 116.2), turned to -90 degrees
- moved C30 45.8 mm to (182.0, 112.4), turned to -90 degrees
- moved R7 41.1 mm to (132.5, 113.3), turned to -90 degrees
- moved J1 37.1 mm to (165.4, 84.5), turned to 0 degrees
- moved R19 35.3 mm to (180.9, 112.4), turned to -90 degrees
- moved R11 32.7 mm to (132.5, 105.4), turned to -90 degrees
- moved R10 29.4 mm to (144.5, 113.3), turned to -90 degrees
- moved C31 24.0 mm to (178.4, 88.0), turned to -90 degrees
- moved R21 20.7 mm to (177.8, 84.2), turned to -90 degrees
- moved C26 19.6 mm to (139.9, 86.2), turned to 180 degrees
- moved R20 15.9 mm to (167.9, 85.0), turned to 90 degrees
- moved D1 11.5 mm to (139.9, 84.3), turned to 180 degrees
- moved U2 9.39 mm to (144.4, 84.8), turned to -90 degrees
- moved R16 7.33 mm to (155.2, 99.2), turned to -90 degrees
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Connections:
- net /SW renamed Net-(U1-SW)
- C14 pad 1: /VCC_VCO -> GND
- C14 pad 2: GND -> /VCC_VCO
- C15 pad 1: /VCC_PLL -> /VCC_DIG
- C16 pad 1: /VCC_PLL -> /VCC_DIG
- C17 pad 1: /VCC_PLL -> /VCC_DIG
- C18 pad 1: /VCC_PLL -> /VCC_DIG
- C19 pad 2: Net-(C19-Pad2) -> Net-(J1-Pin_2)
- C26 pad 1: Net-(C26-Pad1) -> Net-(D1-K)
- C26 pad 2: Net-(C19-Pad2) -> GND
- C30 pad 1: Net-(C26-Pad1) -> Net-(J1-Pin_3)
- D1 pad 1: GND -> Net-(D1-K)
- D1 pad 2: Net-(D1-A) -> /12V
- J1 pad 1: Net-(J1-In) -> Net-(J1-Pin_1)
- J1 pad 2: GND -> Net-(J1-Pin_2)
- R1 pad 1: unconnected-(R1-Pad1) -> /CLK
- R10 pad 1: Net-(R10-Pad1) -> GND
- R10 pad 2: Net-(J1-In) -> Net-(J5-CC2)
- R11 pad 1: Net-(J1-In) -> Net-(D3-A)
- R11 pad 2: /VCC_PLL -> /5V
- R16 pad 1: /Vtune -> /CP
- R16 pad 2: /CP -> /Vtune
- R19 pad 1: Net-(C26-Pad1) -> Net-(J1-Pin_3)
- R2 pad 1: unconnected-(R2-Pad1) -> /DATA
- R20 pad 2: Net-(C26-Pad1) -> Net-(J1-Pin_1)
- R3 pad 1: unconnected-(R3-Pad1) -> /LE
- R7 pad 1: Net-(U1-LD) -> GND
- R7 pad 2: /VCC_PLL -> Net-(J5-CC1)
- U1 pad 25: Net-(U1-LD) -> /LD
- U1 pad 28: /VCC_PLL -> /VCC_DIG
- U1 pad 30: Net-(J1-In) -> /MUX
- U1 pad 32: /VCC_PLL -> /VCC_DIG
- U1 pad 4: unconnected-(U1-CE-Pad4) -> /CE
- U2 pad 1: Net-(U1-LD) -> /5V
- U2 pad 2: /LD -> GND
- U2 pad 3: Net-(J1-In) -> Net-(D1-K)
- U3 pad 4: /VCC_RF -> unconnected-(U3-SENSE-Pad4)
Routing:
- net /5V: track 6.86 -> 163.2 mm, vias 0 -> 12
- net Net-(J1-Pin_3): track 0.00 -> 34.5 mm
- net /LD: track 0.00 -> 28.5 mm, vias 0 -> 4
- net GND: track 36.1 -> 60.8 mm, vias 131 -> 239
- net /RF_EN: track 4.87 -> 26.2 mm, vias 0 -> 2
- net /MUX: track 0.00 -> 21.2 mm
- net /UPDI: track 0.00 -> 15.9 mm
- net /Vtune: track 4.18 -> 19.7 mm, vias 0 -> 4
- net /CE: track 0.00 -> 15.4 mm
- net /TXD_M: track 0.00 -> 14.6 mm
- net /3V3: track 0.00 -> 14.0 mm
- net /VCC_DIG: track 0.00 -> 13.7 mm
- net /CLK: track 0.00 -> 11.1 mm
- net /VCC_TCXO: track 0.00 -> 10.5 mm
- net /VCC_PLL: track 15.2 -> 5.06 mm
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Other:
- board outline added: 60.1 x 39.3 mm
