File: Hardware/Synthesizer.kicad_sch (KiCad schematic)
At the start: 67 parts, among them J1 MUX_OUT, J2 REF_IN, J3 RFOUTA, J4 RFOUTB, T1 HB-TCM2-63WX+, T2 HB-TCM2-63WX+, U2 74LCX07, U3 GM1207ACPZ-3.3, X1 IQXO-70

Commit message: Nearing completion on schematic and layout.  Ready for design review.
Parts:
- removed D1: LOCK, LED_SMD:LED_0402_1005Metric, symbol Device:LED
- removed J1: MUX_OUT, Connector_Coaxial:SMA_Samtec_SMA-J-P-H-ST-EM1_EdgeMount, symbol Connector:Conn_Coaxial
- removed R10, R11, R14, R15: NP, Resistor_SMD:R_0402_1005Metric, symbol Device:R_Small_US
- removed R12, R8, R9: 5K1, Resistor_SMD:R_0402_1005Metric, symbol Device:R_Small_US
- removed R13: 0, Resistor_SMD:R_0402_1005Metric, symbol Device:R_Small_US
- removed R7: OPEN, Resistor_SMD:R_0402_1005Metric, symbol Device:R_Small_US
- removed U2: 74LCX07, Package_SO:TSSOP-14_4.4x5mm_P0.65mm, symbol 74xx:74LCX07
- added C34, C35, C36, C37, C38, C39, C40, C41: 2.2u, Synthesizer:Cap_0402, symbol Device:C
- added C42, C44, C46, C47: .1u, Synthesizer:Cap_0402, symbol Device:C
- added C43, C45: 47p, Synthesizer:Cap_0402, symbol Device:C
- added C48: 6.8u, Capacitor_SMD:C_0603_1608Metric, symbol Device:C
- added D1: D_Schottky, Diode_SMD:D_0603_1608Metric, symbol Device:D_Schottky
- added D2, D4: MM3Z3V6, Diode_SMD:D_SOD-323, symbol Diode:DZ2S036X0L
- added D3, D5: White, LED_SMD:LED_0402_1005Metric, symbol Device:LED
- added D6, D7: Yellow, LED_SMD:LED_0402_1005Metric, symbol Device:LED
- added FB1: FerriteBead_Small, Inductor_SMD:L_0805_2012Metric, symbol Device:FerriteBead_Small
- added J1: REF Select, Connector_PinHeader_2.54mm:PinHeader_1x03_P2.54mm_Vertical, symbol Connector:Conn_01x03_Pin
- added J5: USB-C 2.0 16P, Connector_USB:USB_C_Receptacle_G-Switch_GT-USB-7010ASV, symbol Connector:USB_C_Receptacle_USB2.0_16P
- added J7: Header 1x3, Connector_PinHeader_2.54mm:PinHeader_1x03_P2.54mm_Vertical, symbol Connector:Conn_01x03_Pin
- added J8: Screw_Terminal_01x12, TerminalBlock_TE-Connectivity:TerminalBlock_TE_282834-2_1x02_P2.54mm_Horizontal, symbol Connector:Screw_Terminal_01x02
- added R10, R7: 5K1, Synthesizer:Res_0402, symbol Device:R_US
- added R11, R26, R27, R28, R29, R30: 1K, Synthesizer:Res_0402, symbol Device:R_US
- added R24, R25: 22, Synthesizer:Res_0402, symbol Device:R_US
- added U2: MC78L05_SOT89, Package_TO_SOT_SMD:SOT-89-3, symbol Regulator_Linear:MC78L05_SOT89
- added U4, U5, U6, U7: GM1207ACPZ-3.3, Package_TO_SOT_SMD:SOT-23-5, symbol Synthesizer:GM1207ACPZ-3.3
- added U8: ATtiny1616-M, Package_DFN_QFN:VQFN-20-1EP_3x3mm_P0.4mm_EP1.7x1.7mm, symbol MCU_Microchip_ATtiny:ATtiny1616-M
- added U9: FT231XQ, Package_DFN_QFN:QFN-20-1EP_4x4mm_P0.5mm_EP2.5x2.5mm, symbol Interface_USB:FT231XQ
- C1, C10, C11, C12, C13, C14, C15, C16, C17, C18, C19, C2, C20, C21, C22, C23, C24, C25, C27, C28, C29, C3, C30, C31, C32, C33, C4, C5, C6, C7, C8, C9: footprint Capacitor_SMD:C_0402_1005Metric -> Synthesizer:Cap_0402
- C26: value NP -> 330n 25V; footprint Capacitor_SMD:C_0402_1005Metric -> Capacitor_SMD:C_0603_1608Metric
- R1, R16, R17, R18, R19, R2, R20, R21, R22, R23, R3, R4, R5, R6: footprint Resistor_SMD:R_0402_1005Metric -> Synthesizer:Res_0402
Connections:
- net 5V: now also C35.1, C37.1, C38.1, C40.1, C42.1, C44.1, C47.1, C48.1, D6.2 (A), D7.2 (A), FB1.2, R11.2, U2.1 (OUT), U4.1 (VIN), U4.3 (EN), U5.1 (VIN), U5.3 (EN), U6.1 (VIN), U6.3 (EN), U7.1 (VIN), U7.3 (EN), U8.4 (VCC), U9.12 (VCC)
- net CP: now also R16.1; no longer R16.2
- net GND: now also C14.1, C26.2, C34.2, C35.2, C36.2, C37.2, C38.2, C39.2, C40.2, C41.2, C42.2, C43.2, C44.2, C45.2, C46.2, C47.2, C48.2, D2.2 (A), D3.1 (K), D4.2 (A), J5.A1 (GND), J5.A12 (GND), J5.B1 (GND), J5.B12 (GND), J5.S1 (SHIELD), J8.1 (Pin_1), R10.1, R26.2, R7.1, U2.2 (GND), U4.2 (GND), U5.2 (GND), U6.2 (GND), U7.2 (GND), U8.21 (GND), U8.3 (GND), U9.13 (GND), U9.21 (GND), U9.3 (GND); no longer C14.2
- net LD: now also U1.25 (LD), U8.20 (PA1)
- net RF_EN: now also U8.18 (PC3)
- net VCC_DIG: now also C15.1, C16.1, C17.1, C18.1, U1.28 (VCC_DIG), U1.32 (VDD_SD), C41.1, U7.5 (VOUT)
- net VCC_PLL: now also C34.1, U4.5 (VOUT); no longer C15.1, C16.1, C17.1, C18.1, U1.28 (VCC_DIG), U1.32 (VDD_SD)
- net VCC_RF: no longer U3.4 (SENSE)
- net VCC_TCXO: now also C39.1, U6.5 (VOUT)
- net VCC_VCO: now also C14.2, C36.1, U5.5 (VOUT); no longer C14.1
- net Vtune: now also R16.2; no longer R16.1
- net CLK: now reaches R1.1
- net CLK: now also U8.16 (PC1)
- net MUX: now reaches U1.30 (MUX_OUT)
- net MUX: now also U8.17 (PC2)
- net at C30.1, R19.1: now also J1.3 (Pin_3); no longer C26.1, R20.2
- net LE: now reaches R3.1
- net LE: now also U8.14 (PB0)
- net at C19.2: now also J1.2 (Pin_2); no longer C26.2
- net CE: now reaches U1.4 (CE)
- net CE: now also U8.13 (PB1)
- net DATA: now reaches R2.1
- net DATA: now also U8.15 (PC0)
- net SW: no longer names the net of R17.2, R18.1, U1.5 (SW)
- new net: C26.1, D1.1 (K), U2.3 (IN)
- new net: C45.1, D2.1 (K), J5.A6 (D+), J5.B6 (D+), R25.2
- new net: J5.B5 (CC2), R10.2
- new net: FB1.1, J5.A4 (VBUS), J5.A9 (VBUS), J5.B4 (VBUS), J5.B9 (VBUS)
- new net: D3.2 (A), R11.1
- new net: D5.1 (K), R26.1
- new net: J5.A5 (CC1), R7.2
- new net: C43.1, D4.1 (K), J5.A7 (D-), J5.B7 (D-), R24.2
- new net: D7.1 (K), R28.2
- new net: J1.1 (Pin_1), R20.2
- new net: D6.1 (K), R27.2
- new net 12V: D1.2 (A), J8.2 (Pin_2)
- new net 3V3: C46.1, U9.10 (3V3OUT), U9.11 (~{RESET}), U9.20 (VCCIO)
- new net CTS\: U9.6 (~{CTS})
- new net D+M: R25.1, U9.8 (USBDP)
- new net D-M: R24.1, U9.9 (USBDM)
- new net LED: D5.2 (A), U8.5 (PA4)
- new net RTS\: U9.19 (~{RTS})
- new net RXD_M: R29.2, U8.11 (PB3)
- new net RXD_U: J7.2 (Pin_2), U9.1 (RXD)
- new net RXLED/: R27.1, U9.14 (CBUS1)
- new net SLEEP/: U9.16 (CBUS3)
- new net TXDEN: U9.15 (CBUS0)
- new net TXD_M: J7.3 (Pin_3), U8.12 (PB2)
- new net TXD_U: R29.1, R30.1, U9.17 (TXD)
- new net TXLED/: R28.1, U9.7 (CBUS2)
- new net UPDI: J7.1 (Pin_1), R30.2, U8.19 (~{RESET}/PA0)
- no-connect marks 0 -> 13
Other:
- note added: "CBUS signals use defaults"
- note added: "Comms"
- note added: "Program"
- note added: "What frequency range on output is required? all the way to 6 GHZ? Should board have 1 or 2 RF outputs? How fussy on RFOUT about trace impedance, balance, shielding? Should RFOUT use Balun or just one side to SMA? Should board use SMA or some other RF connector? Should this board be 0.032 thick or made from Rogers material? (make 50 ohm traces narrower) Should board be more than two layers? Layou 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"
- moved on the sheet: C1, C10, C11, C12, C13, C14, C15, C16, C17, C18, C2, C20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
